File: PowerADCs/PowerADCs.kicad_pcb (KiCad board)
At the start: 2 copper layers, 32.5 x 41.5 mm, 28 parts, among them J1 I2C_STANDARDQWIIC, J2 Conn_01x02_Female, J3 Conn_01x10_Female, J4 Conn_01x10_Female, J6 Conn_01x02_Female, J7 Conn_01x02_Female, U1 MCP3428, U2 MCP3428, U3 INA219AxD, U4 SY6280AAC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

Commit message: change ADC's and add seconde qwiic connector
Parts:
- added C3: 0.1uF, Capacitor_SMD:C_0402_1005Metric, F.Cu at (76.8, 84.2)
- added C5: 0.1uF, Capacitor_SMD:C_0402_1005Metric, F.Cu at (77.5, 94.4)
- added J5: I2C_STANDARDQWIIC, Connectors:1X04_1MM_RA, F.Cu at (75.3, 70.8)
- U1, U2: value MCP3428 -> ADS7830; footprint Package_SO:TSSOP-14_4.4x5mm_P0.65mm -> Package_SO:TSSOP-16_4.4x5mm_P0.65mm
- moved U1 1.85 mm to (75.2, 91.0), turned to 0 degrees
- moved U2 1.57 mm to (75.2, 80.3), turned to 0 degrees
Connections:
- J3 pad 1: /CH4 -> /CH8
- J3 pad 2: /CH3 -> /CH7
- J3 pad 3: /CH2 -> /CH6
- J3 pad 4: /CH1 -> /CH5
- J3 pad 5: /CH5 -> /CH4
- J3 pad 6: /CH6 -> /CH3
- J3 pad 7: /CH7 -> /CH2
- J3 pad 8: /CH8 -> /CH1
- J4 pad 1: /CH11 -> /CH16
- J4 pad 2: /CH10 -> /CH15
- J4 pad 3: /CH9 -> /CH14
- J4 pad 4: /CH12 -> /CH13
- J4 pad 5: /CH13 -> /CH12
- J4 pad 6: /CH14 -> /CH11
- J4 pad 7: /CH15 -> /CH10
- J4 pad 8: /CH16 -> /CH9
- U1 pad 10: GND -> Net-(U1-Pad10)
- U1 pad 11: /CH5 -> unconnected-(U1-Pad11)
- U1 pad 12: /CH6 -> GND
- U1 pad 13: /CH7 -> GND
- U1 pad 14: /CH8 -> /I2C_SCL
- U1 pad 5: GND -> /CH5
- U1 pad 6: +3V3 -> /CH6
- U1 pad 7: /I2C_SDA -> /CH7
- U1 pad 8: /I2C_SCL -> /CH8
- U2 pad 10: unconnected-(U2-Pad10) -> Net-(U2-Pad10)
- U2 pad 11: /CH13 -> unconnected-(U2-Pad11)
- U2 pad 12: /CH14 -> +3V3
- U2 pad 13: /CH15 -> GND
- U2 pad 14: /CH16 -> /I2C_SCL
- U2 pad 5: GND -> /CH13
- U2 pad 6: +3V3 -> /CH14
- U2 pad 7: /I2C_SDA -> /CH15
- U2 pad 8: /I2C_SCL -> /CH16
Routing:
- net /I2C_SDA: track 35.4 -> 57.1 mm, vias 2 -> 0
- net +3V3: track 100.6 -> 116.5 mm, vias 5 -> 7
- net /I2C_SCL: track 37.8 -> 47.5 mm, vias 4 -> 2
- net GND: track 22.7 -> 31.4 mm, vias 1 -> 6
- net /CH13: track 10.8 -> 5.08 mm
- net /CH4: track 13.0 -> 8.06 mm
- net /CH12: track 9.26 -> 5.06 mm
- net /CH5: track 12.7 -> 8.72 mm
- net /CH3: track 11.2 -> 7.25 mm
- net /CH14: track 9.22 -> 5.31 mm
- net /CH11: track 9.22 -> 5.31 mm
- net /CH2: track 9.99 -> 6.33 mm
- net Net-(U2-Pad10): track 0.00 -> 3.55 mm
- net Net-(U1-Pad10): track 0.00 -> 3.14 mm
- net /CH8: track 8.11 -> 10.5 mm
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
Commit message: more silkscreen and fix resistor value for current limiter
Parts:
- R3: value 3.4K -> 6.8K
- R5: value 3.4K -> 1.7K
Other:
- board text added: "+"
- board text added: "-"
- board text added: "1"
- board text added: "2"
- board text added: "3"
- board text added: "4"
- board text added: "5"
- board text added: "6"
- board text added: "7"
- board text added: "8"
- board text added: "ADC 1"
- board text added: "ADC 2"
Changed lines of the file:
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@@
   (net 32 "unconnected-(U1-Pad11)")
   (net 33 "unconnected-(U2-Pad11)")
-  (net 34 "Net-(U2-Pad10)")
-  (net 35 "Net-(U1-Pad10)")
+  (net 34 "Net-(C3-Pad1)")
+  (net 35 "Net-(C5-Pad1)")
   (footprint "Capacitor_SMD:C_0402_1005Metric" (layer "F.Cu")
     (at 77.55 94.4)
@@
     (fp_line (start 0.5 -0.25) (end 0.5 0.25) (layer "F.Fab") (width 0.1))
     (pad "1" smd roundrect locked (at -0.48 0) (size 0.56 0.62) (layers "F.Cu" "F.Paste" "F.Mask") (roundrect_rratio 0.25)
-      (net 35 "Net-(U1-Pad10)") (pintype "passive"))
+      (net 35 "Net-(C5-Pad1)") (pintype "passive"))
     (pad "2" smd roundrect locked (at 0.48 0) (size 0.56 0.62) (layers "F.Cu" "F.Paste" "F.Mask") (roundrect_rratio 0.25)
       (net 2 "GND") (pintype "passive"))
@@
       (net 2 "GND") (pinfunction "GND") (pintype "power_in"))
     (pad "10" smd roundrect locked (at 2.8625 1.625) (size 1.475 0.4) (layers "F.Cu" "F.Paste" "F.Mask") (roundrect_rratio 0.25)
-      (net 35 "Net-(U1-Pad10)") (pinfunction "REFin/REFout") (pintype "bidirectional"))
+      (net 35 "Net-(C5-Pad1)") (pinfunction "REFin/REFout") (pintype "bidirectional"))
     (pad "11" smd roundrect locked (at 2.8625 0.975) (size 1.475 0.4) (layers "F.Cu" "F.Paste" "F.Mask") (roundrect_rratio 0.25)
       (net 32 "unconnected-(U1-Pad11)") (pinfunction "COM") (pintype "input"))
@@
       (effects (font (size 0.5 0.5) (thickness 0.1)))
     )
-    (fp_text value "3.4K" (at 0 1.17 90) (layer "F.Fab")
+    (fp_text value "1.7K" (at 0 1.17 90) (layer "F.Fab")
       (effects (font (size 1 1) (thickness 0.15)))
     )
@@
       (net 2 "GND") (pinfunction "GND") (pintype "power_in"))
     (pad "10" smd roundrect locked (at 2.8625 1.625) (size 1.475 0.4) (layers "F.Cu" "F.Paste" "F.Mask") (roundrect_rratio 0.25)
-      (net 34 "Net-(U2-Pad10)") (pinfunction "REFin/REFout") (pintype "bidirectional"))
+      (net 34 "Net-(C3-Pad1)") (pinfunction "REFin/REFout") (pintype "bidirectional"))
     (pad "11" smd roundrect locked (at 2.8625 0.975) (size 1.475 0.4) (layers "F.Cu" "F.Paste" "F.Mask") (roundrect_rratio 0.25)
       (net 33 "unconnected-(U2-Pad11)") (pinfunction "COM") (pintype "input"))
@@
     (property "Sheetname" "")
     (attr smd)
-    (fp_text reference "C3" (at 0 0.9) (layer "F.SilkS")
+    (fp_text reference "C3" (at 1.65 -0.05) (layer "F.SilkS")
       (effects (font (size 0.5 0.5) (thickness 0.1)))
     )
@@
     (fp_line (start -0.5 0.25) (end -0.5 -0.25) (layer "F.Fab") (width 0.1))
     (pad "1" smd roundrect locked (at -0.48 0) (size 0.56 0.62) (layers "F.Cu" "F.Paste" "F.Mask") (roundrect_rratio 0.25)
-      (net 34 "Net-(U2-Pad10)") (pintype "passive"))
+      (net 34 "Net-(C3-Pad1)") (pintype "passive"))
     (pad "2" smd roundrect locked (at 0.48 0) (size 0.56 0.62) (layers "F.Cu" "F.Paste" "F.Mask") (roundrect_rratio 0.25)
       (net 2 "GND") (pintype "passive"))
@@
       (effects (font (size 0.5 0.5) (thickness 0.1)))
     )
-    (fp_text value "3.4K" (at 0 1.17 90) (layer "F.Fab")
+    (fp_text value "6.8K" (at 0 1.17 90) (layer "F.Fab")
       (effects (font (size 1 1) (thickness 0.15)))
     )
@@
   )
   (gr_rect (start 65 107.5) (end 97.5 66) (layer "Edge.Cuts") (width 0.1) (fill none))
+  (gr_text "-" (at 69.3 74.75 90) (layer "F.SilkS")
+    (effects (font (size 0.5 0.5) (thickness 0.1)))
+  )
+  (gr_text "8" (at 69.45 84.7 270) (layer "F.SilkS")
+    (effects (font (size 0.5 0.5) (thickness 0.1)))
+  )
+  (gr_text "-" (at 69.35 90.05 90) (layer "F.SilkS")
+    (effects (font (size 0.5 0.5) (thickness 0.1)))
+  )
   (gr_text "Power&ADC \nV0.1" (at 81.5 74.1) (layer "F.SilkS")
     (effects (font (size 1 1) (thickness 0.2)))
   )
+  (gr_text "7" (at 69.4 83.45 270) (layer "F.SilkS")
+    (effects (font (size 0.5 0.5) (thickness 0.1)))
+  )
+  (gr_text "6" (at 69.45 97.45 270) (layer "F.SilkS")
+    (effects (font (size 0.5 0.5) (thickness 0.1)))
+  )
+  (gr_text "4" (at 69.4 79.7 270) (layer "F.SilkS")
+    (effects (font (size 0.5 0.5) (thickness 0.1)))
+  )
+  (gr_text "3" (at 69.4 78.4 270) (layer "F.SilkS")
+    (effects (font (size 0.5 0.5) (thickness 0.1)))
+  )
   (gr_text "POWER_AUX 3.3V\n+	  -" (at 93.9 82.8 90) (layer "F.SilkS")
     (effects (font (size 0.5 0.5) (thickness 0.1)))
   )
+  (gr_text "6" (at 69.4 82.15 270) (layer "F.SilkS")
+    (effects (font (size 0.5 0.5) (thickness 0.1)))
+  )
+  (gr_text "2" (at 69.45 92.45 270) (layer "F.SilkS")
+    (effects (font (size 0.5 0.5) (thickness 0.1)))
+  )
   (gr_text "2S-4S" (at 78.35 106.25) (layer "F.SilkS")
     (effects (font (size 0.5 0.5) (thickness 0.1)))
   )
+  (gr_text "4" (at 69.45 95 270) (layer "F.SilkS")
+    (effects (font (size 0.5 0.5) (thickness 0.1)))
+  )
   (gr_text "QWIIC" (at 83.4 68.85 270) (layer "F.SilkS")
     (effects (font (size 0.5 0.5) (thickness 0.1)))
   )
+  (gr_text "2" (at 69.4 77.15 270) (layer "F.SilkS")
+    (effects (font (size 0.5 0.5) (thickness 0.1)))
+  )
   (gr_text "Bat\n+	  -" (at 73.6 103.9) (layer "F.SilkS")
     (effects (font (size 0.5 0.5) (thickness 0.1)))
@@
     (effects (font (size 0.5 0.5) (thickness 0.1)))
   )
+  (gr_text "5" (at 69.4 80.95 270) (layer "F.SilkS")
+    (effects (font (size 0.5 0.5) (thickness 0.1)))
+  )
+  (gr_text "3" (at 69.45 93.7 270) (layer "F.SilkS")
+    (effects (font (size 0.5 0.5) (thickness 0.1)))
+  )
+  (gr_text "1" (at 69.45 91.25 270) (layer "F.SilkS")
+    (effects (font (size 0.5 0.5) (thickness 0.1)))
+  )
+  (gr_text "1" (at 69.4 75.95 270) (layer "F.SilkS")
+    (effects (font (size 0.5 0.5) (thickness 0.1)))
+  )
+  (gr_text "+" (at 69.35 88.75 90) (layer "F.SilkS")
+    (effects (font (size 0.5 0.5) (thickness 0.1)))
+  )
+  (gr_text "ADC 1" (at 70.45 94.4 270) (layer "F.SilkS")
+    (effects (font (size 0.5 0.5) (thickness 0.1)))
+  )
+  (gr_text "+" (at 69.3 73.45 90) (layer "F.SilkS")
+    (effects (font (size 0.5 0.5) (thickness 0.1)))
+  )
+  (gr_text "ADC 2" (at 70.4 79.1 270) (layer "F.SilkS")
+    (effects (font (size 0.5 0.5) (thickness 0.1)))
+  )
   (gr_text "QWIIC" (at 79.65 68.85 270) (layer "F.SilkS")
     (effects (font (size 0.5 0.5) (thickness 0.1)))
   )
+  (gr_text "5" (at 69.45 96.25 270) (layer "F.SilkS")
+    (effects (font (size 0.5 0.5) (thickness 0.1)))
+  )
+  (gr_text "8" (at 69.5 100 270) (layer "F.SilkS")
+    (effects (font (size 0.5 0.5) (thickness 0.1)))
+  )
+  (gr_text "7" (at 69.45 98.75 270) (layer "F.SilkS")
+    (effects (font (size 0.5 0.5) (thickness 0.1)))
+  )
